File: hardware/emonTH V2.0.2.sch (EAGLE design)
At the start: 47 parts, among them J1 1X2-3.5MM, J2 1X2-3.5MM, J3 1X2-3.5MM, Q1 16Mhz, Q2 DS18B20, U1 LTC3525ESC6-3.3TRMPBF, U1_MLF ATMEGA168MLF, U1_TQFP ATMEGA328P, U2 SI7021

Commit message: update portmap & sch + brd img
Other:
- note added: "D16 DHT22 data"
- note removed: "D17 DHT22 data"
Changed lines of the file:
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@@
 <text x="104.14" y="367.665" size="3.81" layer="91">RFM12B
 RFM1269CW</text>
-<text x="2.54" y="233.68" size="1.778" layer="91">D17
+<text x="2.54" y="233.68" size="1.778" layer="91">D16
 DHT22 data</text>
 <text x="106.68" y="292.1" size="1.778" layer="91">Si7020 / HTU21D Temperature &amp; Humidity </text>
